Commit message: kukaiiwa_slide_xacro

File: kukaiiwa_slide_xacro/urdf/slide.xacro (robot description, xacro)
@@ -1,5 +1,60 @@
 <?xml version="1.0"?>
-<robot name="kukaiiwa" xmlns:xacro="http://wiki.ros.org/xacro">
-    <xacro:include filename="$(find kukaiiwa_xacro)/urdf/kukaiiwa_macro.xacro" />
+<robot name="slide" xmlns:xacro="http://wiki.ros.org/xacro">
+    <xacro:include filename="$(find kukaiiwa_slide_xacro)/urdf/slide_macro.xacro" />
+	<xacro:include filename="$(find kukaiiwa_slide_xacro)/urdf/kukaiiwa_macro.xacro" />
+		<!-- slide -->
+		<xacro:slide_macro
+			slide_name="slide">
+		</xacro:slide_macro>
+		<!-- first joint wheel -->
+		<xacro:wheel_to_plane_joint
+			name="front_whell_dx_joint"
+			parent="slide"
+			child="front_whell_dx">
+			<origin xyz="8 7.5 -3.5" />
+		</xacro:wheel_to_plane_joint>
+		<!-- first wheel-->
+		<xacro:wheel name="front_whell_dx">
+			<origin xyz="0 0 0" rpy="0 1.57 0"/>
+		</xacro:wheel>
+		<!-- second joint wheel -->
+		<xacro:wheel_to_plane_joint
+			name="front_whell_sx_joint"
+			parent="slide"
+			child="front_whell_sx">
+			<origin xyz="-8 7.5 -3.5" />
+		</xacro:wheel_to_plane_joint>
+		<!-- second wheel-->
+		<xacro:wheel name="front_whell_sx">
+			<origin xyz="0 0 0" rpy="0 1.57 0"/>
+		</xacro:wheel>
+		<!-- third joint wheel-->
+		<xacro:wheel_to_plane_joint
+			name="rear_whell_dx_joint"
+			parent="slide"
+			child="rear_whell_dx">
+			<origin xyz="8 -7.5 -3.5" />
+		</xacro:wheel_to_plane_joint>
+		<!-- third wheel-->
+		<xacro:wheel name="rear_whell_dx">
+			<origin xyz="0 0 0" rpy="0 1.57 0"/>
+		</xacro:wheel>
+		<!-- fourh joint wheel-->
+		<xacro:wheel_to_plane_joint
+			name="rear_whell_sx_joint"
+			parent="slide"
+			child="rear_whell_sx">
+			<origin xyz="-8 -7.5 -3.5" />
+		</xacro:wheel_to_plane_joint>
+		<!-- fourth wheel-->
+		<xacro:wheel name="rear_whell_sx">
+			<origin xyz="0 0 0" rpy="0 1.57 0"/>
+		</xacro:wheel>
+		<!-- robot_to_slide_joint-->
+		<joint name="robot_to_slide" type="fixed">
+			<parent link="slide" />
+			<child link="base_link" />
+			<origin xyz="0 0 1.5"/>
+		</joint>
 		<!-- base link -->
 		<xacro:base_link_macro
@@ -21,5 +76,5 @@
 				<cylinder length="20" radius="5"/>
 			</geometry>
-			<origin xyz="0 0 12.5" rpy="0 0 0"/>
+			<origin xyz="0 0 15" rpy="0 0 0"/>
 		</xacro:kukaiiwa_link>
 		<!-- second joint -->
@@ -29,5 +84,5 @@
 			parent="first_link"
 			child="second_link">
-			<origin xyz="0 0 17.5"/>
+			<origin xyz="0 0 20"/>
 			<axis xyz="1 0 0"/>
 			<limit effort="176" velocity="1.96" lower="-2.09" upper="2.09" />

File: kukaiiwa_slide_xacro/urdf/slide_generated.urdf (robot description, URDF)
Before this commit: robot kukaiiwa, 8 links, 7 joints
Links:
- added link front_whell_dx, mass 1; collision cylinder length=2 radius=2; visual cylinder length=2 radius=2
- added link front_whell_sx, mass 1; collision cylinder length=2 radius=2; visual cylinder length=2 radius=2
- added link rear_whell_dx, mass 1; collision cylinder length=2 radius=2; visual cylinder length=2 radius=2
- added link rear_whell_sx, mass 1; collision cylinder length=2 radius=2; visual cylinder length=2 radius=2
- added link slide, mass 1; collision box size=3 20 20; visual box size=3 20 20
Joints:
- added joint front_whell_dx_joint: type revolute, parent slide, child front_whell_dx, origin xyz=8 7.5 -3.5, axis 1 0 0, limit lower=3.1415 upper=-3.1415 effort=1 velocity=2.5
- added joint front_whell_sx_joint: type revolute, parent slide, child front_whell_sx, origin xyz=-8 7.5 -3.5, axis 1 0 0, limit lower=3.1415 upper=-3.1415 effort=1 velocity=2.5
- added joint rear_whell_dx_joint: type revolute, parent slide, child rear_whell_dx, origin xyz=8 -7.5 -3.5, axis 1 0 0, limit lower=3.1415 upper=-3.1415 effort=1 velocity=2.5
- added joint rear_whell_sx_joint: type revolute, parent slide, child rear_whell_sx, origin xyz=-8 -7.5 -3.5, axis 1 0 0, limit lower=3.1415 upper=-3.1415 effort=1 velocity=2.5
- added joint robot_to_slide: type fixed, parent slide, child base_link, origin xyz=0 0 1.5
- joint second_joint: origin xyz=0 0 17.5 -> xyz=0 0 20

File: kukaiiwa_slide_xacro/urdf/slide_macro.xacro (robot description, xacro)
@@ -1,20 +1,20 @@
 <?xml version="1.0"?>
-<robot name="kukaiwaa_macro" xmlns:xacro="http://wiki.ros.org/xacro">
-	<xacro:macro name="base_link_macro" params="base_link_name">
-		<link name="${base_link_name}">
+<robot name="slide_macro" xmlns:xacro="http://wiki.ros.org/xacro">
+	<xacro:macro name="slide_macro" params="slide_name">
+		<link name="${slide_name}">
 			<visual>
 				<geometry>
-					<cylinder length="5" radius="8"/>
+					<box size="3 20 20"/>
 				</geometry>
-				<origin rpy="0 0 0" xyz="0 0 0"/>
-				<material name="yellow">
-					<color rgba="1 1 0 1"/>
+				<origin rpy="0 1.57 0" xyz="0 0 0"/>
+				<material name="red">
+					<color rgba="1 0 0 1"/>
 				</material>
 			</visual>
 			<collision>
 				<geometry>
-					<cylinder length="5" radius="8"/>
+					<box size="3 20 20"/>
 				</geometry>
-				<origin rpy="0 0 0" xyz="0 0 0"/>
+				<origin rpy="0 1.57 0" xyz="0 0 0"/>
 			</collision>
 			<inertial>
@@ -24,25 +24,29 @@
 		</link>
 	</xacro:macro>
-	<xacro:macro name="kukaiiwa_joint" params="name type parent child *origin *axis *limit">
-		<joint name="${name}" type="${type}">
+	<xacro:macro name="wheel_to_plane_joint" params="name parent child *origin">
+		<joint name="${name}" type="revolute">
 			<parent link="${parent}" />
 			<child link="${child}" />
 	   		<xacro:insert_block name="origin" />
-			<xacro:insert_block name="axis" />
-			<xacro:insert_block name="limit"/>
-			<dynamics damping="50" friction="1"/>
+			<axis xyz="1 0 0"/>
+			<limit effort="1" velocity="2.5" upper="-3.1415" lower="3.1415"/>
+			<dynamics damping="10" friction="1"/>
 		</joint>
 	</xacro:macro>
-	<xacro:macro name="kukaiiwa_link" params="name *geometry *origin">
+	<xacro:macro name="wheel" params="name *origin">
 		<link name="${name}">
 			<visual>
-				<xacro:insert_block name="geometry" />
+				<geometry>
+					<cylinder length="2" radius="2"/>
+				</geometry>
 				<xacro:insert_block name="origin" />
-				<material name="red">
+				<material name="blue">
 				  <color rgba="0 0 1 1"/>
 				</material>
 			</visual>
 			<collision>
-				<xacro:insert_block name="geometry" />
+				<geometry>
+					<cylinder length="2" radius="2"/>
+				</geometry>
 				<xacro:insert_block name="origin" />
 			</collision>
